File: _KiCad/water-leak-sms-alarm.kicad_sch (KiCad schematic)
At the start: 32 parts, among them Q1 NTR4101PT1G, Q2 PMV16XNR, Q3 PMV16XNR, Q4 PMV16XNR, SW1 TEST, SW2 BYPASS, U1 MCP1700x-120xxTO, U2 mini_esp32, U3 SIM800L-CORE

Commit message: Update water-leak-sms-alarm.kicad_sch
Parts:
- added R5: 680K, Resistor_SMD:R_0805_2012Metric_Pad1.20x1.40mm_HandSolder, symbol Device:R
- renumbered R9 to R10, R10 to R11, R11 to R12, R5 to R6, R6 to R7, R7 to R8, R8 to R9
Connections:
- net GND: now also R5.1
- net at Q2.2 (G), Q3.1 (D), R1.1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: now also R5.2
Changed lines of the file:
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@@
 	)
 	(junction
+		(at 66.04 92.71)
+		(diameter 0)
+		(color 0 0 0 0)
+	)
+	(junction
 		(at 63.5 147.32)
 		(diameter 0)
@@
 	(wire
 		(pts
+			(xy 80.01 80.01) (xy 80.01 82.55)
+		)
+		(stroke
+			(width 0)
+			(type default)
+		)
+	)
+	(wire
+		(pts
 			(xy 130.81 80.01) (xy 143.51 80.01)
 		)
@@
 	(wire
 		(pts
+			(xy 66.04 92.71) (xy 80.01 92.71)
+		)
+		(stroke
+			(width 0)
+			(type default)
+		)
+	)
+	(wire
+		(pts
 			(xy 124.46 40.64) (xy 124.46 45.72)
 		)
@@
 	(wire
 		(pts
-			(xy 66.04 85.09) (xy 66.04 95.25)
-		)
-		(stroke
-			(width 0)
-			(type default)
-		)
-	)
-	(wire
-		(pts
 			(xy 100.33 147.32) (xy 63.5 147.32)
 		)
@@
 	(wire
 		(pts
+			(xy 66.04 85.09) (xy 66.04 92.71)
+		)
+		(stroke
+			(width 0)
+			(type default)
+		)
+	)
+	(wire
+		(pts
 			(xy 142.24 130.81) (xy 143.51 130.81)
 		)
@@
 	(wire
 		(pts
+			(xy 66.04 92.71) (xy 66.04 95.25)
+		)
+		(stroke
+			(width 0)
+			(type default)
+		)
+	)
+	(wire
+		(pts
 			(xy 121.92 45.72) (xy 124.46 45.72)
 		)
@@
 		)
 	)
+	(wire
+		(pts
+			(xy 80.01 92.71) (xy 80.01 90.17)
+		)
+		(stroke
+			(width 0)
+			(type default)
+		)
+	)
 	(polyline
 		(pts
@@
 		(on_board yes)
 		(dnp no)
-		(property "Reference" "R5"
+		(property "Reference" "R6"
 			(at 135.382 85.344 0)
 			(effects
@@
 			(project "water-leak-sms-alarm"
 				(path "/60aaadb6-22e4-4148-b1e3-ea6c0e67e0dd"
-					(reference "R5")
+					(reference "R6")
 					(unit 1)
 				)
@@
 	(symbol
 		(lib_id "Device:R")
+		(at 80.01 86.36 180)
+		(unit 1)
+		(exclude_from_sim no)
+		(in_bom yes)
+		(on_board yes)
+		(dnp no)
+		(property "Reference" "R5"
+			(at 75.184 85.09 0)
+			(effects
+				(font
+					(size 1.27 1.27)
+				)
+			)
+		)
+		(property "Value" "680K"
+			(at 75.438 87.122 0)
+			(effects
+				(font
+					(size 1.27 1.27)
+				)
+			)
+		)
+		(property "Footprint" "Resistor_SMD:R_0805_2012Metric_Pad1.20x1.40mm_HandSolder"
+			(at 81.788 86.36 90)
+			(effects
+				(font
+					(size 1.27 1.27)
+				)
+				(hide yes)
+			)
+		)
+		(property "Datasheet" "https://www.mouser.se/datasheet/2/315/AOA0000C307-1149632.pdf"
+			(at 80.01 86.36 0)
+			(effects
+				(font
+					(size 1.27 1.27)
+				)
+				(hide yes)
+			)
+		)
+		(property "Description" "ERA-6AEB104V "
+			(at 80.01 86.36 0)
+			(effects
+				(font
+					(size 1.27 1.27)
+				)
+				(hide yes)
+			)
+		)
+		(pin "1"
+		)
+		(pin "2"
+		)
+		(instances
+			(project "water-leak-sms-alarm"
+				(path "/60aaadb6-22e4-4148-b1e3-ea6c0e67e0dd"
+					(reference "R5")
+					(unit 1)
+				)
+			)
+		)
+	)
+	(symbol
+		(lib_id "Device:R")
 		(at 63.5 153.67 180)
 		(unit 1)
@@
 		(on_board yes)
 		(dnp no)
-		(property "Reference" "R9"
+		(property "Reference" "R10"
 			(at 68.072 152.146 0)
 			(effects
@@
 			(project "water-leak-sms-alarm"
 				(path "/60aaadb6-22e4-4148-b1e3-ea6c0e67e0dd"
-					(reference "R9")
+					(reference "R10")
 					(unit 1)
 				)
@@
 		(on_board yes)
 		(dnp no)
-		(property "Reference" "R8"
+		(property "Reference" "R9"
 			(at 41.656 150.114 90)
 			(effects
@@
 			(project "water-leak-sms-alarm"
 				(path "/60aaadb6-22e4-4148-b1e3-ea6c0e67e0dd"
-					(reference "R8")
+					(reference "R9")
 					(unit 1)
 				)
@@
 		(on_board yes)
 		(dnp no)
-		(property "Reference" "R11"
+		(property "Reference" "R12"
 			(at 243.332 143.764 0)
 			(effects
@@
 			(project "water-leak-sms-alarm"
 				(path "/60aaadb6-22e4-4148-b1e3-ea6c0e67e0dd"
-					(reference "R11")
+					(reference "R12")
 					(unit 1)
 				)
@@
 		(on_board yes)
 		(dnp no)
-		(property "Reference" "R6"
+		(property "Reference" "R7"
 			(at 85.344 120.65 0)
 			(effects
@@
 			(project "water-leak-sms-alarm"
 				(path "/60aaadb6-22e4-4148-b1e3-ea6c0e67e0dd"
-					(reference "R6")
+					(reference "R7")
 					(unit 1)
 				)
@@
 		(on_board yes)
 		(dnp no)
-		(property "Reference" "R10"
+		(property "Reference" "R11"
 			(at 46.99 182.118 90)
 			(effects
@@
 			(project "water-leak-sms-alarm"
 				(path "/60aaadb6-22e4-4148-b1e3-ea6c0e67e0dd"
-					(reference "R10")
+					(reference "R11")
 					(unit 1)
 				)
@@
 		(on_board yes)
 		(dnp no)
-		(property "Reference" "R7"
+		(property "Reference" "R8"
 			(at 85.344 130.302 0)
 			(effects
@@
 			(project "water-leak-sms-alarm"
 				(path "/60aaadb6-22e4-4148-b1e3-ea6c0e67e0dd"
-					(reference "R7")
+					(reference "R8")
 					(unit 1)
 				)

Commit message: Update water-leak-sms-alarm.kicad_sch
Parts:
- R5: value 680K -> 300K
Changed lines of the file:
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@@
 			)
 		)
-		(property "Value" "680K"
+		(property "Value" "300K"
 			(at 75.438 87.122 0)
 			(effects
